Commit message: add a rgb camera to cable joint world

File: cable_joint_description/urdf/cable_joint.gazebo.xacro (robot description, xacro)
@@ -1,4 +1,50 @@
 <?xml version="1.0"?>
 <robot>
+  <!-- camera -->
+  <gazebo reference="link_optical">
+    <sensor type="camera" name="camera1">
+      <update_rate>30.0</update_rate>
+      <camera name="rgb">
+        <horizontal_fov>1.3962634</horizontal_fov>
+        <image>
+          <width>800</width>
+          <height>800</height>
+          <format>R8G8B8</format>
+        </image>
+        <clip>
+          <near>0.02</near>
+          <far>300</far>
+        </clip>
+        <noise>
+          <type>gaussian</type>
+          <!-- Noise is sampled independently per pixel on each frame.
+               That pixel's noise value is added to each of its color
+               channels, which at that point lie in the range [0,1]. -->
+          <mean>0.0</mean>
+          <stddev>0.007</stddev>
+        </noise>
+      </camera>
+      <plugin name="camera_controller" filename="libgazebo_ros_camera.so">
+        <alwaysOn>true</alwaysOn>
+        <updateRate>0.0</updateRate>
+        <cameraName>cable_joint/rgb_camera</cameraName>
+        <imageTopicName>image_raw</imageTopicName>
+        <cameraInfoTopicName>camera_info</cameraInfoTopicName>
+        <frameName>link_optical</frameName>
+        <hackBaseline>0.07</hackBaseline>
+        <distortionK1>0.0</distortionK1>
+        <distortionK2>0.0</distortionK2>
+        <distortionK3>0.0</distortionK3>
+        <distortionT1>0.0</distortionT1>
+        <distortionT2>0.0</distortionT2>
+      </plugin>
+    </sensor>
+  </gazebo>
+  <gazebo reference="link_lens">
+    <material>Gazebo/Black</material>
+  </gazebo>
+  <gazebo reference="link_camera_body">
+    <material>Gazebo/Red</material>
+  </gazebo>
   <gazebo reference="link_base">
     <material>Gazebo/Black</material>
@@ -26,5 +72,5 @@
   </gazebo>
   <gazebo reference="link_disc">
-    <material>Gazebo/White</material>
+    <material>Gazebo/Grey</material>
   </gazebo>
   <gazebo reference="link_cube_northeast">

File: cable_joint_description/urdf/cable_joint.urdf.xacro (robot description, xacro)
@@ -3,4 +3,5 @@
   <!-- Constants for robot dimensions -->
   <xacro:property name="PI" value="3.1415926535897931"/>
+  <xacro:property name="body_length" value="0.02" /> <!-- Size of square 'camera' box -->
   <!-- Import all Gazebo-customization elements, including Gazebo colors -->
   <xacro:include filename="$(find gazebo_rl)/cable_joint_description/urdf/cable_joint.gazebo.xacro" />
@@ -36,4 +37,69 @@
     </inertial>
   </link>
+  <joint name="joint_world_camerabody" type="revolute">
+    <origin rpy="0 0 ${PI/2}" xyz="0 -0.5 ${body_length/2}"/>
+    <parent link="world"/>
+    <child link="link_camera_body"/>
+    <limit effort="0" lower="0" upper="0" velocity="0"/>
+    <axis rpy="0 0 0" xyz="0 0 1"/>
+  </joint>
+  <link name="link_camera_body">
+    <collision>
+      <origin rpy="0 0 0" xyz="0 -0.5 0"/>
+      <geometry>
+        <box size="${body_length} ${body_length*2} ${body_length*2}"/>
+      </geometry>
+    </collision>
+    <visual>
+      <origin rpy="0 0 0" xyz="0 0 0"/>
+      <geometry>
+        <box size="${body_length} ${body_length*2} ${body_length*2}"/>
+      </geometry>
+      <material name="red"/>
+    </visual>
+    <inertial>
+      <mass value="0.1"/>
+      <origin rpy="0 0 0" xyz="0 0 0"/>
+      <inertia ixx="1e-6" ixy="0" ixz="0" iyy="1e-6" iyz="0" izz="1e-6"/>
+    </inertial>
+  </link>
+  <joint name="joint_camerabody_lens" type="revolute">
+    <origin rpy="0 ${PI/2} 0" xyz="${body_length/2+body_length/16} 0 0"/>
+    <parent link="link_camera_body"/>
+    <child link="link_lens"/>
+    <limit effort="0" lower="0" upper="0" velocity="0"/>
+    <axis rpy="0 0 0" xyz="0 0 1"/>
+  </joint>
+  <link name="link_lens">
+    <collision>
+      <origin rpy="0 0 0" xyz="0 -0.5 0"/>
+      <geometry>
+        <cylinder length="${body_length/8}" radius="${body_length/2}"/>
+      </geometry>
+    </collision>
+    <visual>
+      <origin rpy="0 0 0" xyz="0 0 0"/>
+      <geometry>
+        <cylinder length="${body_length/8}" radius="${body_length/2}"/>
+      </geometry>
+      <material name="black"/>
+    </visual>
+    <inertial>
+      <mass value="0.01"/>
+      <origin rpy="0 0 0" xyz="0 0 0"/>
+      <inertia ixx="1e-6" ixy="0" ixz="0" iyy="1e-6" iyz="0" izz="1e-6"/>
+    </inertial>
+  </link>
+  <!-- In order to correctly display camera -->
+   <joint name="camera_optical_joint" type="fixed">
+    <!-- these values have to be these values otherwise the gazebo camera
+        image won't be aligned properly with the frame it is supposedly
+        originating from -->
+    <origin xyz="0 0 0" rpy="${-PI/2} ${-PI/2} ${PI/2}"/>
+    <parent link="link_lens"/>
+    <child link="link_optical"/>
+  </joint>
+  <link name="link_optical">
+  </link>
   <joint name="joint_base_lowersupport" type="revolute">
     <origin rpy="0 0 0" xyz="0 0 0"/>

Commit message: add force plugin to cable joint

File: cable_joint_description/urdf/cable_joint.gazebo.xacro (robot description, xacro)
@@ -40,4 +40,22 @@
       </plugin>
     </sensor>
+  </gazebo>
+  <gazebo>
+    <plugin filename="libgazebo_ros_force.so" name="gazebo_ros_force">
+      <bodyName>link_cube_northeast</bodyName>
+      <topicName>/force_northeast</topicName>
+    </plugin>
+    <plugin filename="libgazebo_ros_force.so" name="gazebo_ros_force">
+      <bodyName>link_cube_northwest</bodyName>
+      <topicName>/force_northwest</topicName>
+    </plugin>
+    <plugin filename="libgazebo_ros_force.so" name="gazebo_ros_force">
+      <bodyName>link_cube_southeast</bodyName>
+      <topicName>/force_southeast</topicName>
+    </plugin>
+    <plugin filename="libgazebo_ros_force.so" name="gazebo_ros_force">
+      <bodyName>link_cube_southwest</bodyName>
+      <topicName>/force_southwest</topicName>
+    </plugin>
   </gazebo>
   <gazebo reference="link_lens">

File: cable_joint_description/urdf/cable_joint.urdf.xacro (robot description, xacro)
@@ -111,5 +111,5 @@
       <origin rpy="0 0 0" xyz="0 0 0.07"/>
       <geometry>
-        <cylinder length="0.14" radius="0.01"/>
+        <cylinder length="0.14" radius="0.015"/>
       </geometry>
     </collision>
@@ -117,5 +117,5 @@
       <origin rpy="0 0 0" xyz="0 0 0.07"/>
       <geometry>
-        <cylinder length="0.14" radius="0.01"/>
+        <cylinder length="0.14" radius="0.015"/>
       </geometry>
       <material name="grey"/>
@@ -124,11 +124,13 @@
       <mass value="100"/>
       <origin rpy="0 0 0" xyz="0 0 0"/>
-      <inertia ixx="0.2533" ixy="0" ixz="0" iyy="0.2533" iyz="0" izz="0.5236"/>
-    </inertial>
-  </link>
-  <joint name="joint_base_pinwest" type="fixed">
+      <inertia ixx="0.1" ixy="0" ixz="0" iyy="0.1" iyz="0" izz="0.1"/>
+    </inertial>
+  </link>
+  <joint name="joint_base_pinwest" type="revolute">
     <parent link="link_base"/>
     <child link="link_pin_west"/>
     <origin rpy="0 0 0" xyz="-0.1 0 0.01"/>
+    <limit effort="0" lower="0" upper="0" velocity="0"/>
+    <axis rpy="0 0 0" xyz="0 0 1"/>
   </joint>
   <link name="link_pin_west">
@@ -149,11 +151,13 @@
       <mass value="1"/>
       <origin rpy="0 0 0" xyz="0 0 0"/>
-      <inertia ixx="0.0002" ixy="0" ixz="0" iyy="0.0002" iyz="0" izz="0.0002"/>
-    </inertial>
-  </link>
-  <joint name="joint_base_pineast" type="fixed">
+      <inertia ixx="1e-4" ixy="0" ixz="0" iyy="1e-4" iyz="0" izz="1e-4"/>
+    </inertial>
+  </link>
+  <joint name="joint_base_pineast" type="revolute">
     <parent link="link_base"/>
     <child link="link_pin_east"/>
     <origin rpy="0 0 0" xyz="0.1 0 0.01"/>
+    <limit effort="0" lower="0" upper="0" velocity="0"/>
+    <axis rpy="0 0 0" xyz="0 0 1"/>
   </joint>
   <link name="link_pin_east">
@@ -174,5 +178,5 @@
       <mass value="1"/>
       <origin rpy="0 0 0" xyz="0 0 0"/>
-      <inertia ixx="0.0002" ixy="0" ixz="0" iyy="0.0002" iyz="0" izz="0.0002"/>
+      <inertia ixx="1e-4" ixy="0" ixz="0" iyy="1e-4" iyz="0" izz="1e-4"/>
     </inertial>
   </link>
@@ -180,7 +184,7 @@
     <parent link="link_lower_support"/>
     <child link="link_ball_roll"/>
-    <origin rpy="${PI/2} 0 0" xyz="0 0 0.14"/>
-    <axis xyz="0 0 1"/>
-    <limit effort="100" velocity="1000" lower="${-PI/2}" upper="${PI/2}"/>
+    <origin rpy="0 0 0" xyz="0 0 0.14"/>
+    <axis xyz="1 0 0"/>
+    <limit effort="10" velocity="${PI*2}" lower="${-4*PI/9}" upper="${4*PI/9}"/>
   </joint>
   <link name="link_ball_roll">
@@ -199,7 +203,7 @@
     </visual>
     <inertial>
-      <mass value="0.5"/>
-      <origin rpy="0 0 0" xyz="0 0 0"/>
-      <inertia ixx="0.000001" ixy="0" ixz="0" iyy="0.000001" iyz="0" izz="0.000001"/>
+      <mass value="0.1"/>
+      <origin rpy="0 0 0" xyz="0 0 0"/>
+      <inertia ixx="1e-8" ixy="0" ixz="0" iyy="1e-8" iyz="0" izz="1e-8"/>
     </inertial>
   </link>
@@ -207,7 +211,7 @@
     <parent link="link_ball_roll"/>
     <child link="link_ball_pitch"/>
-    <origin rpy="0 ${PI/2} 0" xyz="0 0 0"/>
-    <axis xyz="0 0 1"/>
-    <limit effort="100" velocity="1000" lower="${-PI/2}" upper="${PI/2}"/>
+    <origin rpy="0 0 0" xyz="0 0 0"/>
+    <axis xyz="0 1 0"/>
+    <limit effort="10" velocity="${PI*2}" lower="${-4*PI/9}" upper="${4*PI/9}"/>
   </joint>
   <link name="link_ball_pitch">
@@ -226,7 +230,7 @@
     </visual>
     <inertial>
-      <mass value="0.5"/>
-      <origin rpy="0 0 0" xyz="0 0 0"/>
-      <inertia ixx="0.000001" ixy="0" ixz="0" iyy="0.000001" iyz="0" izz="0.000001"/>
+      <mass value="0.1"/>
+      <origin rpy="0 0 0" xyz="0 0 0"/>
+      <inertia ixx="1e-8" ixy="0" ixz="0" iyy="1e-8" iyz="0" izz="1e-8"/>
     </inertial>
   </link>
@@ -234,7 +238,7 @@
     <parent link="link_ball_pitch"/>
     <child link="link_ball_yaw"/>
-    <origin rpy="${-PI/2} 0 0" xyz="0 0 0"/>
+    <origin rpy="0 0 0" xyz="0 0 0"/>
     <axis xyz="0 0 1"/>
-    <limit effort="100" velocity="1000" lower="${-PI/8}" upper="${PI/8}"/>
+    <limit effort="10" velocity="${PI*2}" lower="${-PI/8}" upper="${PI/8}"/>
   </joint>
   <link name="link_ball_yaw">
@@ -255,11 +259,11 @@
       <mass value="1"/>
       <origin rpy="0 0 0" xyz="0 0 0"/>
-      <inertia ixx="0.00016" ixy="0" ixz="0" iyy="0.00016" iyz="0" izz="0.00016"/>
+      <inertia ixx="1e-6" ixy="0" ixz="0" iyy="1e-6" iyz="0" izz="1e-6"/>
     </inertial>
   </link>
   <joint name="joint_ballyaw_uppersupport" type="revolute">
-    <origin rpy="0 0 0" xyz="0 0 0"/>
-    <limit effort="0" lower="0" upper="0" velocity="0"/>
-    <axis rpy="0 0 0" xyz="0 0 1"/>
+    <origin rpy="0 0 0" xyz="0 0 0.03"/>
+    <limit effort="0" lower="0" upper="0" velocity="0"/>
+    <axis xyz="0 0 1"/>
     <parent link="link_ball_yaw"/>
     <child link="link_upper_support"/>
@@ -267,5 +271,5 @@
   <link name="link_upper_support">
     <collision>
-      <origin rpy="0 0 0" xyz="0 0 0.02"/>
+      <origin rpy="0 0 0" xyz="0 0 0"/>
       <geometry>
         <cylinder length="0.04" radius="0.01"/>
@@ -273,5 +277,5 @@
     </collision>
     <visual>
-      <origin rpy="0 0 0" xyz="0 0 0.02"/>
+      <origin rpy="0 0 0" xyz="0 0 0"/>
       <geometry>
         <cylinder length="0.04" radius="0.01"/>
@@ -280,13 +284,13 @@
     </visual>
     <inertial>
-      <mass value="0.001"/>
-      <origin rpy="0 0 0" xyz="0 0 0.02"/>
-      <inertia ixx="0.0000002" ixy="0" ixz="0" iyy="0.0000002" iyz="0" izz="0.0000001"/>
+      <mass value="1e-5"/>
+      <origin rpy="0 0 0" xyz="0 0 0"/>
+      <inertia ixx="1e-8" ixy="0" ixz="0" iyy="1e-8" iyz="0" izz="1e-8"/>
     </inertial>
   </link>
   <joint name="joint_uppersupport_disc" type="revolute">
-    <origin rpy="0 0 ${-PI/2}" xyz="0 0 0.04"/>
-    <limit effort="0" lower="0" upper="0" velocity="0"/>
-    <axis rpy="0 0 0" xyz="0 0 1"/>
+    <origin rpy="0 0 0" xyz="0 0 0.02"/>
+    <limit effort="0" lower="0" upper="0" velocity="0"/>
+    <axis xyz="0 0 1"/>
     <parent link="link_upper_support"/>
     <child link="link_disc"/>
@@ -307,13 +311,15 @@
     </visual>
     <inertial>
-      <mass value="0.001"/>
-      <origin rpy="0 0 0" xyz="0 0 0.02"/>
-      <inertia ixx="0.0000025" ixy="0" ixz="0" iyy="0.0000025" iyz="0" izz="0.000005"/>
-    </inertial>
-  </link>
-  <joint name="joint_disc_cubenortheast" type="fixed">
+      <mass value="0.0001"/>
+      <origin rpy="0 0 0" xyz="0 0 0"/>
+      <inertia ixx="1e-6" ixy="0" ixz="0" iyy="1e-6" iyz="0" izz="1e-6"/>
+    </inertial>
+  </link>
+  <joint name="joint_disc_cubenortheast" type="revolute">
     <parent link="link_disc"/>
     <child link="link_cube_northeast"/>
     <origin rpy="0 0 0" xyz="0.0707 0.0707 0"/>
+    <limit effort="0" lower="0" upper="0" velocity="0"/>
+    <axis rpy="0 0 0" xyz="0 0 1"/>
   </joint>
   <link name="link_cube_northeast">
@@ -332,13 +338,15 @@
     </visual>
     <inertial>
-      <mass value="0.0001"/>
-      <origin rpy="0 0 0" xyz="0 0 0"/>
-      <inertia ixx="0.00000001" ixy="0" ixz="0" iyy="0.00000001" iyz="0" izz="0.00000001"/>
-    </inertial>
-  </link>
-  <joint name="joint_disc_cubenorthwest" type="fixed">
+      <mass value="1e-5"/>
+      <origin rpy="0 0 0" xyz="0 0 0"/>
+      <inertia ixx="1e-8" ixy="0" ixz="0" iyy="1e-8" iyz="0" izz="1e-8"/>
+    </inertial>
+  </link>
+  <joint name="joint_disc_cubenorthwest" type="revolute">
     <parent link="link_disc"/>
     <child link="link_cube_northwest"/>
     <origin rpy="0 0 0" xyz="-0.0707 0.0707 0"/>
+    <limit effort="0" lower="0" upper="0" velocity="0"/>
+    <axis rpy="0 0 0" xyz="0 0 1"/>
   </joint>
   <link name="link_cube_northwest">
@@ -357,13 +365,15 @@
     </visual>
     <inertial>
-      <mass value="0.0001"/>
-      <origin rpy="0 0 0" xyz="0 0 0"/>
-      <inertia ixx="0.00000001" ixy="0" ixz="0" iyy="0.00000001" iyz="0" izz="0.00000001"/>
-    </inertial>
-  </link>
-    <joint name="joint_disc_cubesouthwest" type="fixed">
+      <mass value="1e-5"/>
+      <origin rpy="0 0 0" xyz="0 0 0"/>
+      <inertia ixx="1e-8" ixy="0" ixz="0" iyy="1e-8" iyz="0" izz="1e-8"/>
+    </inertial>
+  </link>
+  <joint name="joint_disc_cubesouthwest" type="revolute">
     <parent link="link_disc"/>
     <child link="link_cube_southwest"/>
     <origin rpy="0 0 0" xyz="-0.0707 -0.0707 0"/>
+    <limit effort="0" lower="0" upper="0" velocity="0"/>
+    <axis rpy="0 0 0" xyz="0 0 1"/>
   </joint>
   <link name="link_cube_southwest">
@@ -382,13 +392,15 @@
     </visual>
     <inertial>
-      <mass value="0.0001"/>
-      <origin rpy="0 0 0" xyz="0 0 0"/>
-      <inertia ixx="0.00000001" ixy="0" ixz="0" iyy="0.00000001" iyz="0" izz="0.00000001"/>
-    </inertial>
-  </link>
-  <joint name="joint_disc_cubesoutheast" type="fixed">
+      <mass value="1e-5"/>
+      <origin rpy="0 0 0" xyz="0 0 0"/>
+      <inertia ixx="1e-8" ixy="0" ixz="0" iyy="1e-8" iyz="0" izz="1e-8"/>
+    </inertial>
+  </link>
+  <joint name="joint_disc_cubesoutheast" type="revolute">
     <parent link="link_disc"/>
     <child link="link_cube_southeast"/>
     <origin rpy="0 0 0" xyz="0.0707 -0.0707 0"/>
+    <limit effort="0" lower="0" upper="0" velocity="0"/>
+    <axis rpy="0 0 0" xyz="0 0 1"/>
   </joint>
   <link name="link_cube_southeast">
@@ -407,7 +419,7 @@
     </visual>
     <inertial>
-      <mass value="0.0001"/>
-      <origin rpy="0 0 0" xyz="0 0 0"/>
-      <inertia ixx="0.00000001" ixy="0" ixz="0" iyy="0.00000001" iyz="0" izz="0.00000001"/>
+      <mass value="1e-5"/>
+      <origin rpy="0 0 0" xyz="0 0 0"/>
+      <inertia ixx="1e-8" ixy="0" ixz="0" iyy="1e-8" iyz="0" izz="1e-8"/>
     </inertial>
   </link>
